Commit message: 修改：     locomotion/model_test.py 	修改：     locomotion/wheel_legged_env.py 	修改：     locomotion/wheel_legged_eval.py 	修改：     locomotion/wheel_legged_train.py

File: assets/urdf/nz/urdf/nz.urdf (robot description, URDF)
Before this commit: robot nz, 9 links, 8 joints
Joints:
- joint left_thigh_joint: limit lower=-2.530729 upper=0 effort=40 velocity=0 -> lower=-0.785399 upper=0.785399 effort=40 velocity=0
- joint right_thigh_joint: limit lower=-2.530729 upper=0 effort=40 velocity=0 -> lower=-0.785399 upper=0.785399 effort=40 velocity=0
