Commit message: 速度很好 原因：电机扭矩不够

File: assets/urdf/nz2/urdf/nz2.urdf (robot description, URDF)
Before this commit: robot nz2, 9 links, 8 joints
Links:
- removed link right_calf_Link
- removed link right_wheel_Link
- added link right_calf_link, mass 0.347648888154323; collision mesh filename=package://nz2/meshes/right_calf_link.STL; visual mesh filename=package://nz2/meshes/right_calf_link.STL
- added link right_wheel_link, mass 0.440514867448173; collision mesh filename=package://nz2/meshes/right_wheel_link.STL; visual mesh filename=package://nz2/meshes/right_wheel_link.STL
Joints:
- joint right_calf_joint: child right_calf_Link -> right_calf_link
- joint right_wheel_joint: child right_wheel_Link -> right_wheel_link; parent right_calf_Link -> right_calf_link
